Commit message: Cleaned up and packaged nodes

File: urdf/boat.urdf.xacro (robot description, xacro)
@@ -19,7 +19,7 @@
  </visual>
     <collision>
-    <origin xyz="0 0 0" rpy="0 0 0" />
-     <geometry>
-       <mesh filename="package://boat/meshes/BoatHull.STL" scale="0.001 0.001 0.001"/>
+    <origin xyz="0 0 2" rpy="${PI/2} 0 ${PI/2}" />
+    <geometry>
+     <mesh filename="package://boat/meshes/BoatHull.STL" scale="0.01 0.01 0.01"/>
     </geometry>
     </collision>
@@ -46,7 +46,7 @@
  </visual>
     <collision>
-    <origin xyz="0 0 0" rpy="0 0 0" />
-     <geometry>
-       <mesh filename="package://boat/meshes/hullstl.STL" scale="0.001 0.001 0.001"/>
+    <origin xyz="0 0 0" rpy="${PI/2} 0 ${PI/2}" />
+    <geometry>
+     <mesh filename="package://boat/meshes/hullstl.STL" scale="0.01 0.01 0.01"/>
     </geometry>
     </collision>
@@ -76,7 +76,7 @@
  </visual>
     <collision>
-    <origin xyz="0 0 0" rpy="0 0 0" />
-     <geometry>
-       <mesh filename="package://boat/meshes/PropHousingCase1.STL" scale="0.001 0.001 0.001"/>
+    <origin xyz="0 0 0" rpy="${PI/2} 0 ${3*PI/2}" />
+    <geometry>
+     <mesh filename="package://boat/meshes/PropHousingCase1.STL" scale="0.01 0.01 0.01"/>
     </geometry>
     </collision>
@@ -98,7 +98,7 @@
  </visual>
     <collision>
-    <origin xyz="0 0 0" rpy="0 0 0" />
-     <geometry>
-       <mesh filename="package://boat/meshes/Servo Turning.STL" scale="0.001 0.001 0.001"/>
+    <origin xyz="1.43 0 0" rpy="${PI/2} 0 ${PI/2}" />
+    <geometry>
+     <mesh filename="package://boat/meshes/Servo Turning.STL" scale="0.01 0.01 0.01"/>
     </geometry>
     </collision>
@@ -127,7 +127,7 @@
  </visual>
     <collision>
-    <origin xyz="0 0 0" rpy="0 0 ${PI}" />
-     <geometry>
-       <mesh filename="package://boat/meshes/7297K180.STL" scale="0.001 0.001 0.001"/>
+    <origin xyz="0 -0.14 -0.14" rpy="0 0 ${PI/2}" />
+    <geometry>
+     <mesh filename="package://boat/meshes/7297K180.STL" scale="0.01 0.01 0.01"/>
     </geometry>
     </collision>
@@ -157,7 +157,7 @@
  </visual>
     <collision>
-    <origin xyz="0 0 0" rpy="0 0 0" />
-     <geometry>
-       <mesh filename="package://boat/meshes/Shaft.STL" scale="0.001 0.001 0.001"/>
+    <origin xyz="2.04 0.205 0" rpy="${PI/2} 0 ${PI/2+0.1}" />
+    <geometry>
+     <mesh filename="package://boat/meshes/Shaft.STL" scale="0.01 0.01 0.01"/>
     </geometry>
     </collision>
@@ -187,7 +187,7 @@
  </visual>
     <collision>
-    <origin xyz="0 0 0" rpy="0 0 0" />
-     <geometry>
-       <mesh filename="package://boat/meshes/PropPiece.STL" scale="0.001 0.001 0.001"/>
+    <origin xyz="2.04 0.195 1.155" rpy="${PI/2} 0 ${PI/2+0.1}" />
+    <geometry>
+     <mesh filename="package://boat/meshes/PropPiece.STL" scale="0.01 0.01 0.01"/>
     </geometry>
     </collision>
